File: PCB Files/Spooky-Season-Distributor/Spooky-Season-Distributor.kicad_sch (KiCad schematic)
At the start: 18 parts, among them J1 Raspberry_Pi_4, J2 Power IN 12v 3.3A, J3 Conn_01x08, M1 Motor_Servo, U1 LM2576T-ADJ, U2 LM2576T-ADJ

Commit message: Finished Routing
This should be most of the PCB routing done, now onto the case!
Parts:
- R2: value 3.16 kΩ, 1% -> 3.90 kΩ, 1%
Changed lines of the file:
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@@
+	)
+	(junction
+		(at 138.43 22.86)
+		(diameter 0)
+		(color 0 0 0 0)
 	)
 	(junction
@@
 	(wire
 		(pts
+			(xy 138.43 25.4) (xy 138.43 22.86)
+		)
+		(stroke
+			(width 0)
+			(type default)
+		)
+	)
+	(wire
+		(pts
 			(xy 113.03 31.75) (xy 113.03 43.18)
 		)
@@
 	(global_label "GND"
 		(shape input)
-		(at 138.43 22.86 270)
+		(at 138.43 25.4 270)
 		(fields_autoplaced yes)
 		(effects
@@
 		)
 		(property "Intersheetrefs" "${INTERSHEET_REFS}"
-			(at 138.43 29.7157 90)
+			(at 138.43 32.2557 90)
 			(hide yes)
 			(show_name no)
@@
 			)
 		)
-		(property "Value" "3.16 kΩ, 1%"
+		(property "Value" "3.90 kΩ, 1%"
 			(at 113.03 40.6399 0)
 			(show_name no)
@@
 					(unit 1)
 				)
+			)
+		)
+	)
+	(symbol
+		(lib_id "power:GND")
+		(at 138.43 22.86 90)
+		(unit 1)
+		(body_style 1)
+		(exclude_from_sim no)
+		(in_bom yes)
+		(on_board yes)
+		(in_pos_files yes)
+		(dnp no)
+		(fields_autoplaced yes)
+		(property "Reference" "#PWR01"
+			(at 144.78 22.86 0)
+			(hide yes)
+			(show_name no)
+			(do_not_autoplace no)
+			(effects
+				(font
+					(size 1.27 1.27)
+				)
+			)
+		)
+		(property "Value" "GND"
+			(at 142.24 22.8599 90)
+			(show_name no)
+			(do_not_autoplace no)
+			(effects
+				(font
+					(size 1.27 1.27)
+				)
+				(justify right)
+			)
+		)
+		(property "Footprint" ""
+			(at 138.43 22.86 0)
+			(hide yes)
+			(show_name no)
+			(do_not_autoplace no)
+			(effects
+				(font
+					(size 1.27 1.27)
+				)
+			)
+		)
+		(property "Datasheet" ""
+			(at 138.43 22.86 0)
+			(hide yes)
+			(show_name no)
+			(do_not_autoplace no)
+			(effects
+				(font
+					(size 1.27 1.27)
+				)
+			)
+		)
+		(property "Description" "Power symbol creates a global label with name \"GND\" , ground"
+			(at 138.43 22.86 0)
+			(hide yes)
+			(show_name no)
+			(do_not_autoplace no)
+			(effects
+				(font
+					(size 1.27 1.27)
+				)
+			)
+		)
+		(pin "1"
+		)
+		(instances
+			(project "Spooky-Season-Distributor"
+				(path "/3013b8d5-9f57-4305-8605-3d7a05968388"
+					(reference "#PWR01")
+					(unit 1)
+				)
