File: PCB Files/Spooky-Season-Distributor/Spooky-Season-Distributor.kicad_pcb (KiCad board)
At the start: 2 copper layers, 159 x 194 mm, 18 parts, among them J1 Raspberry_Pi_4, J2 Power IN 12v 3.3A, J3 Conn_01x08, M1 Motor_Servo, U1 LM2576T-ADJ, U2 LM2576T-ADJ

Commit message: Fixing some DRC issues
Parts:
- U1, U2: footprint Package_TO_SOT_THT:TO-220-5_Vertical -> Assorted Kicad Footprints:TO-220-5_Vertical
Other:
- board text added: "Created by FastTurtle for Hackclub Halflife Thnka you Hackclub!"
- board text added: "Sppoky Season Spirit Distibutor"
- board text added: "Square here"
